Commit message: [ARM-54] Mise à jour des sous-modules dans un fork AltranArmada

File: ardupilot_sitl_gazebo_plugin/urdf/sensors/generic_camera.urdf.xacro (robot description, xacro)
@@ -21,5 +21,5 @@
           <origin xyz="0 0 0" rpy="0 0 0" />
           <geometry>
-            <mesh filename="model://board_camera/meshes/board_camera.dae"/>
+            <mesh filename="file://$(find ardupilot_sitl_gazebo_plugin)/meshes/meshes_sensors/board_camera/meshes/board_camera.dae"/>
           <!--<box size="0.001 0.001 0.001" />-->
           </geometry>

File: ardupilot_sitl_gazebo_plugin/urdf/sensors/lidar_sensor.urdf.xacro (robot description, xacro)
@@ -1,5 +1,5 @@
 <?xml version="1.0"?>
 <robot xmlns:xacro="http://ros.org/wiki/xacro">
-  <xacro:macro name="lidar_sensor" params="name parent *origin ros_topic update_rate min_range max_range field_of_view_horizontal field_of_view_vertical ray_count_horizontal ray_count_vertical sensor_mesh">
+  <xacro:macro name="lidar_sensor" params="name parent *origin update_rate min_range max_range field_of_view_horizontal field_of_view_vertical ray_count_horizontal ray_count_vertical sensor_mesh_base_1 sensor_mesh_base_2 sensor_mesh_scan">
     <joint name="${name}_joint" type="fixed">
       <xacro:insert_block name="origin" />
@@ -14,10 +14,31 @@
       </inertial>
       <visual>
-        <origin xyz="0 0 0" rpy="0 0 0" />
+        <origin xyz="0 0 -0.03" rpy="0 0 0" />
         <geometry>
           <!--<box size="0.01 0.01 0.01" /> -->
           <!-- <mesh filename="package://rotors_description/meshes/sonar_sensor/max_sonar_ez4.dae"/> -->
-           <!--<mesh filename="package://ardupilot_sitl_gazebo_plugin/meshes/${sensor_mesh}"/>-->
-         <!-- <mesh filename="package://ardupilot_sitl_gazebo_plugin/meshes/lidar_lite_v2/meshes/lidar_lite_v2.dae"/> -->
+          <!--<mesh filename="package://ardupilot_sitl_gazebo_plugin/meshes/${sensor_mesh}"/>-->
+           <mesh filename="file://${sensor_mesh_base_1}"/>
+         <!-- <mesh filename="package://ardupilot_sitl_gazebo_plugin/meshes/meshes_sensor/lidar_lite_v2/meshes/lidar_lite_v2.dae"/> -->
+        </geometry>
+      </visual>
+      <visual>
+        <origin xyz="0 0 -0.03" rpy="0 0 0" />
+        <geometry>
+          <!--<box size="0.01 0.01 0.01" /> -->
+          <!-- <mesh filename="package://rotors_description/meshes/sonar_sensor/max_sonar_ez4.dae"/> -->
+          <!--<mesh filename="package://ardupilot_sitl_gazebo_plugin/meshes/${sensor_mesh}"/>-->
+           <mesh filename="file://${sensor_mesh_base_2}"/>
+         <!-- <mesh filename="package://ardupilot_sitl_gazebo_plugin/meshes/meshes_sensor/lidar_lite_v2/meshes/lidar_lite_v2.dae"/> -->
+        </geometry>
+      </visual>
+      <visual>
+        <origin xyz="0 0 -0.03" rpy="0 0 0" />
+        <geometry>
+          <!--<box size="0.01 0.01 0.01" /> -->
+          <!-- <mesh filename="package://rotors_description/meshes/sonar_sensor/max_sonar_ez4.dae"/> -->
+          <!--<mesh filename="package://ardupilot_sitl_gazebo_plugin/meshes/${sensor_mesh}"/>-->
+           <mesh filename="file://${sensor_mesh_scan}"/>
+         <!-- <mesh filename="package://ardupilot_sitl_gazebo_plugin/meshes/meshes_sensor/lidar_lite_v2/meshes/lidar_lite_v2.dae"/> -->
         </geometry>
       </visual>
@@ -56,9 +77,10 @@
           </range>
         </ray>
-        <plugin name="gazebo_ros_${name}_controller" filename="librotors_gazebo_sonar_plugin.so">
-          <gaussianNoise>0.005</gaussianNoise>
-          <topicName>${ros_topic}</topicName>
-          <frameId>${name}_link</frameId>
-        </plugin>
+	<plugin name="gazebo_ros_${name}_controller" filename="libgazebo_ros_laser.so">
+	<!--  <plugin name="gazebo_ros_${name}_controller" filename="libgazebo_ros_gpu_laser.so"> -->
+          <topicName>/scan</topicName>
+          <!-- <frameName>scan_link</frameName> -->
+	  <frameName>lidar_link</frameName>
+	</plugin>
       </sensor>
     </gazebo>

File: ardupilot_sitl_gazebo_plugin/urdf/sensors/sonar_sensor.urdf.xacro (robot description, xacro)
@@ -35,5 +35,5 @@
         <update_rate>${update_rate}</update_rate>
         <pose>0 0 0 0 0 0</pose>
-        <visualize>false</visualize>
+        <visualize>true</visualize>
         <ray>
           <scan>
@@ -63,5 +63,5 @@
         </plugin>
       </sensor>
-    </gazebo>
+   </gazebo>
   </xacro:macro>
 </robot>
